Commit message: add ros2_control control systems, both jazzy and humble compatible
On branch main
Your branch is up to date with 'origin/main'.

Changes to be committed:
	modified:   src/mobile_robot_bringup/config/gz_bridge.yaml
	new file:   src/mobile_robot_bringup/config/ign_bridge.yaml
	modified:   src/mobile_robot_bringup/launch/mobile_robot_gz_sim.launch.py
	modified:   src/mobile_robot_bringup/launch/mobile_robot_gz_sim.launch.xml
	modified:   src/mobile_robot_bringup/package.xml
	new file:   src/mobile_robot_controller/CMakeLists.txt
	new file:   src/mobile_robot_controller/config/mobile_robot_controllers.yaml
	new file:   src/mobile_robot_controller/launch/controller.launch.py
	new file:   src/mobile_robot_controller/launch/controller.launch.xml
	new file:   src/mobile_robot_controller/package.xml
	modified:   src/mobile_robot_description/package.xml
	modified:   src/mobile_robot_description/urdf/camera.urdf.xacro
	modified:   src/mobile_robot_description/urdf/common_properties.urdf.xacro
	modified:   src/mobile_robot_description/urdf/depth_camera.urdf.xacro
	modified:   src/mobile_robot_description/urdf/imu.urdf.xacro
	modified:   src/mobile_robot_description/urdf/lidar.urdf.xacro
	modified:   src/mobile_robot_description/urdf/mobile_base_1.urdf.xacro
	modified:   src/mobile_robot_description/urdf/mobile_base_1_gazebo.urdf.xacro
	new file:   src/mobile_robot_description/urdf/mobile_base_1_ros2_control.urdf.xacro
	modified:   src/mobile_robot_description/urdf/mobile_robot.urdf.xacro

File: src/mobile_robot_description/urdf/camera.urdf.xacro (robot description, xacro)
@@ -14,5 +14,5 @@
                 <box size="${camera_length} ${camera_width} ${camera_height}" />
             </geometry>
-            <material name="gray" />
+            <material name="dark_gray" />
             <origin xyz="0 0 0" rpy="0 0 0" />
         </visual>

File: src/mobile_robot_description/urdf/common_properties.urdf.xacro (robot description, xacro)
@@ -12,4 +12,7 @@
     <material name="gray" >
         <color rgba="0.8 0.8 0.8 1" />
+    </material>
+    <material name="dark_gray">
+        <color rgba="0.3 0.3 0.3 1" />
     </material>
     <xacro:macro name="box_inertial" params="mass size origin_xyz origin_rpy" >

File: src/mobile_robot_description/urdf/depth_camera.urdf.xacro (robot description, xacro)
@@ -14,5 +14,5 @@
                 <box size="${depth_camera_length} ${depth_camera_width} ${depth_camera_height}" />
             </geometry>
-            <material name="gray" />
+            <material name="dark_gray" />
             <origin xyz="0 0 0" rpy="0 0 0" />
         </visual>

File: src/mobile_robot_description/urdf/imu.urdf.xacro (robot description, xacro)
@@ -6,4 +6,5 @@
                 <box size="0.05 0.05 0.05"/>
             </geometry>
+            <material name="dark_gray" />
         </visual>
         <collision>

File: src/mobile_robot_description/urdf/lidar.urdf.xacro (robot description, xacro)
@@ -6,4 +6,5 @@
                 <cylinder length="0.05" radius="0.025"/>
             </geometry>
+            <material name="dark_gray" />
         </visual>
         <collision>

File: src/mobile_robot_description/urdf/mobile_base_1.urdf.xacro (robot description, xacro)
@@ -52,5 +52,7 @@
         <origin xyz="0 0 ${base_height / 2.0 + wheel_radius}" rpy="0 0 0"/>
     </joint>
-    <link name="base_link" />
+    <link name="base_link" >
+        <xacro:box_inertial mass="1.0" size="${base_length} ${base_width} ${base_height}" origin_xyz="0 0 0" origin_rpy="0 0 0"/>
+    </link>
     <joint name="base_left_joint" type="fixed">
         <parent link="base_link"/>

File: src/mobile_robot_description/urdf/mobile_base_1_gazebo.urdf.xacro (robot description, xacro)
@@ -17,24 +17,69 @@
         <mu2 value="0.1"/>
     </gazebo>
-    <gazebo>
-        <plugin filename="gz-sim-diff-drive-system" name="gz::sim::systems::DiffDrive">
-            <left_joint>base_left_wheel_joint</left_joint>
-            <right_joint>base_right_wheel_joint</right_joint>
-            <wheel_separation>${base_width - (wheel_length + epsilon)}</wheel_separation>
-            <wheel_radius>${wheel_radius}</wheel_radius>
-            <odom_publish_frequency>50</odom_publish_frequency>
-            <frame_id>odom</frame_id>
-            <child_frame_id>base_footprint</child_frame_id>
-            <topic>/cmd_vel</topic>
-            <odom_topic>/odometry</odom_topic>
-            <tf_topic>/tf</tf_topic>
-        </plugin>
-    </gazebo>
-    <gazebo>
-        <plugin filename="gz-sim-joint-state-publisher-system" name="gz::sim::systems::JointStatePublisher">
-            <!-- <joint_name>base_left_wheel_joint</joint_name>
-            <joint_name>base_right_wheel_joint</joint_name> -->
-            <topic>/joint_states</topic>
-        </plugin>
-    </gazebo>
+    <xacro:if value="$(arg is_gz)" >
+        <!-- <gazebo>
+            <plugin filename="gz-sim-diff-drive-system" name="gz::sim::systems::DiffDrive">
+                <left_joint>base_left_wheel_joint</left_joint>
+                <right_joint>base_right_wheel_joint</right_joint>
+                <wheel_separation>${base_width - (wheel_length + epsilon)}</wheel_separation>
+                <wheel_radius>${wheel_radius}</wheel_radius>
+                <odom_publish_frequency>50</odom_publish_frequency>
+                <frame_id>odom</frame_id>
+                <child_frame_id>base_footprint</child_frame_id>
+                <topic>/cmd_vel</topic>
+                <odom_topic>/odometry</odom_topic>
+                <tf_topic>/tf</tf_topic>
+            </plugin>
+        </gazebo> -->
+        <!-- <gazebo>
+            <plugin filename="gz-sim-joint-state-publisher-system" name="gz::sim::systems::JointStatePublisher">
+                <joint_name>base_left_wheel_joint</joint_name>
+                <joint_name>base_right_wheel_joint</joint_name>
+                <topic>/joint_states</topic>
+            </plugin>
+        </gazebo> -->
+        <gazebo>
+            <plugin filename="gz_ros2_control-system" name="gz_ros2_control::GazeboSimROS2ControlPlugin" >
+                <parameters>$(find mobile_robot_controller)/config/mobile_robot_controllers.yaml</parameters>
+                <controller_manager_node_name>controller_manager</controller_manager_node_name>
+                <ros>
+                    <remapping>/diff_drive_base_controller/cmd_vel:=/cmd_vel</remapping>
+                    <remapping>/diff_drive_base_controller/odom:=/odom</remapping>
+                </ros>
+            </plugin>
+        </gazebo>
+    </xacro:if>
+    <xacro:unless value="$(arg is_gz)">
+        <!-- <gazebo>
+            <plugin filename="ignition-gazebo-diff-drive-system" name="ignition::gazebo::systems::DiffDrive">
+                <left_joint>base_left_wheel_joint</left_joint>
+                <right_joint>base_right_wheel_joint</right_joint>
+                <wheel_separation>${base_width - (wheel_length + epsilon)}</wheel_separation>
+                <wheel_radius>${wheel_radius}</wheel_radius>
+                <odom_publish_frequency>50</odom_publish_frequency>
+                <frame_id>odom</frame_id>
+                <child_frame_id>base_footprint</child_frame_id>
+                <topic>/cmd_vel</topic>
+                <odom_topic>/odometry</odom_topic>
+                <tf_topic>/tf</tf_topic>
+            </plugin>
+        </gazebo> -->
+        <!-- <gazebo>
+            <plugin filename="ignition-gazebo-joint-state-publisher-system" name="ignition::gazebo::systems::JointStatePublisher">
+                <joint_name>base_left_wheel_joint</joint_name>
+                <joint_name>base_right_wheel_joint</joint_name>
+                <topic>/joint_states</topic>
+            </plugin>
+        </gazebo> -->
+        <gazebo>
+            <plugin filename="ign_ros2_control-system" name="ign_ros2_control::IgnitionROS2ControlPlugin" >
+                <parameters>$(find mobile_robot_controller)/config/mobile_robot_controllers.yaml</parameters>
+                <controller_manager_node_name>controller_manager</controller_manager_node_name>
+                <ros>
+                    <remapping>/diff_drive_base_controller/cmd_vel:=/cmd_vel</remapping>
+                    <remapping>/diff_drive_base_controller/odom:=/odom</remapping>
+                </ros>
+            </plugin>
+        </gazebo>
+    </xacro:unless>
 </robot>

File: src/mobile_robot_description/urdf/mobile_robot.urdf.xacro (robot description, xacro)
@@ -1,7 +1,9 @@
 <?xml version="1.0" encoding="UTF-8"?>
 <robot name="mobile_robot" xmlns:xacro="http://www.ros.org/wiki/xacro">
+    <xacro:arg name="is_gz" default="true" />
     <xacro:include filename="common_properties.urdf.xacro"/>
     <xacro:include filename="mobile_base_1.urdf.xacro" />
     <xacro:include filename="mobile_base_1_gazebo.urdf.xacro" />
+    <xacro:include filename="mobile_base_1_ros2_control.urdf.xacro" />
     <xacro:include filename="camera.urdf.xacro" />
     <xacro:include filename="depth_camera.urdf.xacro" />
