Commit message: add AMR meshes
On branch main
Your branch is up to date with 'origin/main'.

Changes to be committed:
	modified:   src/mobile_robot_bringup/launch/mobile_robot_gz_sim.launch.py
	modified:   src/mobile_robot_controller/config/mobile_robot_controllers.yaml
	modified:   src/mobile_robot_controller/launch/controller.launch.py
	modified:   src/mobile_robot_description/CMakeLists.txt
	modified:   src/mobile_robot_description/launch/display.launch.py
	new file:   src/mobile_robot_description/meshes/chasis.STL
	new file:   src/mobile_robot_description/meshes/wheel.STL
	new file:   src/mobile_robot_description/meshes/zed.STL
	new file:   src/mobile_robot_description/urdf/camera_1.urdf.xacro
	renamed:    src/mobile_robot_description/urdf/camera.urdf.xacro -> src/mobile_robot_description/urdf/camera_2.urdf.xacro
	modified:   src/mobile_robot_description/urdf/common_properties.urdf.xacro
	new file:   src/mobile_robot_description/urdf/depth_camera_1.urdf.xacro
	renamed:    src/mobile_robot_description/urdf/depth_camera.urdf.xacro -> src/mobile_robot_description/urdf/depth_camera_2.urdf.xacro
	renamed:    src/mobile_robot_description/urdf/imu.urdf.xacro -> src/mobile_robot_description/urdf/imu_1.urdf.xacro
	new file:   src/mobile_robot_description/urdf/imu_2.urdf.xacro
	modified:   src/mobile_robot_description/urdf/lidar.urdf.xacro
	new file:   src/mobile_robot_description/urdf/lidar_1.urdf.xacro
	new file:   src/mobile_robot_description/urdf/lidar_2.urdf.xacro
	new file:   src/mobile_robot_description/urdf/mobile_base.urdf.xacro
	modified:   src/mobile_robot_description/urdf/mobile_base_1.urdf.xacro
	modified:   src/mobile_robot_description/urdf/mobile_base_2.urdf.xacro
	modified:   src/mobile_robot_description/urdf/mobile_base_3.urdf.xacro
	modified:   src/mobile_robot_description/urdf/mobile_robot.urdf.xacro
	new file:   src/mobile_robot_description/urdf/zed_camera.urdf.xacro
	new file:   src/mobile_robot_description/urdf/zed_imu.urdf.xacro
	modified:   src/mobile_robot_description/worlds/Depot/model.sdf

File: src/mobile_robot_description/urdf/common_properties.urdf.xacro (robot description, xacro)
@@ -15,4 +15,10 @@
     <material name="dark_gray">
         <color rgba="0.3 0.3 0.3 1" />
+    </material>
+    <material name="chassis_grey">
+        <color rgba="0.5 0.5 0.5 1.0"/>
+    </material>
+    <material name="wheel_grey">
+        <color rgba="0.5 0.5 0.5 1.0"/>
     </material>
     <xacro:macro name="box_inertial" params="mass size origin_xyz origin_rpy" >

File: src/mobile_robot_description/urdf/lidar.urdf.xacro (robot description, xacro)
@@ -1,23 +1,27 @@
 <?xml version="1.0" encoding="UTF-8" ?>
 <robot xmlns:xacro="http://www.ros.org/wiki/xacro" >
+    <xacro:property name="lidar_length" value="0.03" />
+    <xacro:property name="lidar_radius" value="0.05" />
+    <joint name="top_lidar_joint" type="fixed">
+        <parent link="base_link"/>
+        <child link="lidar_link"/>
+        <origin xyz="0.0 0.0 ${base_height}" rpy="0.0 0.0 0.0"/>
+    </joint>
     <link name="lidar_link">
         <visual>
+            <origin xyz="0.0 0.0 0.0" rpy="0.0 0.0 0.0"/>
             <geometry>
-                <cylinder length="0.05" radius="0.025"/>
+                <cylinder radius="${lidar_radius}" length="${lidar_length}"/>
             </geometry>
-            <material name="dark_gray" />
+            <material name="red" />
         </visual>
         <collision>
+            <origin xyz="0.0 0.0 0.0" rpy="0.0 0.0 0.0"/>
             <geometry>
-                <cylinder length="0.05" radius="0.025"/>
+                <cylinder radius="${lidar_radius}" length="${lidar_length}"/>
             </geometry>
         </collision>
-        <xacro:cylinder_inertial mass="0.03" length="0.05" radius="0.025" origin_xyz="0 0 0" origin_rpy="0 0 0" />
+        <xacro:cylinder_inertial mass="0.03" length="${lidar_length}" radius="${lidar_radius}" origin_xyz="0 0 0" origin_rpy="0 0 0" />
     </link>
-    <joint name="top_lidar_joint" type="fixed">
-        <parent link="base_top_link"/>
-        <child link="lidar_link"/>
-        <origin xyz="0 0 ${(boundary_thickness + 0.05) / 2.0}" rpy="0 0 0"/>
-    </joint>
     <gazebo reference="lidar_link">
         <sensor type="gpu_lidar" name="gpu_lidar">

File: src/mobile_robot_description/urdf/mobile_base_1.urdf.xacro (robot description, xacro)
@@ -1,9 +1,7 @@
 <?xml version="1.0" encoding="UTF-8" ?>
 <robot xmlns:xacro="http://www.ros.org/wiki/xacro">
-    <xacro:property name="epsilon" value="0.002"/>
     <xacro:property name="base_length" value="0.6"/>
     <xacro:property name="base_width" value="0.4"/>
     <xacro:property name="base_height" value="0.2"/>
-    <xacro:property name="boundary_thickness" value="0.01"/>
     <xacro:property name="wheel_radius" value="${base_height / 2.0}"/>
     <xacro:property name="wheel_length" value="${wheel_radius / 2.0}"/>
@@ -20,5 +18,4 @@
             <collision>
                 <geometry>
-                    <!-- <cylinder radius="${wheel_radius}" length="${wheel_length}"/> -->
                     <sphere radius="${wheel_radius}" />
                 </geometry>
@@ -52,16 +49,8 @@
         <origin xyz="0 0 ${base_height / 2.0 + wheel_radius}" rpy="0 0 0"/>
     </joint>
-    <link name="base_link" >
-        <xacro:box_inertial mass="1.0" size="${base_length} ${base_width} ${base_height}" origin_xyz="0 0 0" origin_rpy="0 0 0"/>
-    </link>
-    <joint name="base_left_joint" type="fixed">
-        <parent link="base_link"/>
-        <child link="base_left_link"/>
-        <origin xyz="0 ${+ (base_width + boundary_thickness) / 2.0} 0" rpy="0 0 0"/>
-    </joint>
-    <link name="base_left_link">
+    <link name="base_link">
         <visual>
             <geometry>
-                <box size="${base_length + 2.0 * boundary_thickness} ${boundary_thickness} ${base_height + 2.0 * boundary_thickness}"/>
+                <box size="${base_length} ${base_width} ${base_height}"/>
             </geometry>
             <material name="green"/>
@@ -70,98 +59,14 @@
         <collision>
             <geometry>
-                <box size="${base_length + 2.0 * boundary_thickness} ${boundary_thickness} ${base_height + 2.0 * boundary_thickness}"/>
+                <box size="${base_length} ${base_width} ${base_height}"/>
             </geometry>
             <origin xyz="0 0 0" rpy="0 0 0"/>
         </collision>
-        <xacro:box_inertial mass="1.0" size="${base_length + 2.0 * boundary_thickness} ${boundary_thickness} ${base_height + 2.0 * boundary_thickness}" origin_xyz="0 0 0" origin_rpy="0 0 0"/>
-    </link>
-    <joint name="base_right_joint" type="fixed">
-        <parent link="base_link"/>
-        <child link="base_right_link"/>
-        <origin xyz="0 ${- (base_width + boundary_thickness) / 2.0} 0" rpy="0 0 0"/>
-    </joint>
-    <link name="base_right_link">
-        <visual>
-            <geometry>
-                <box size="${base_length + 2.0 * boundary_thickness} ${boundary_thickness} ${base_height + 2.0 * boundary_thickness}"/>
-            </geometry>
-            <material name="green"/>
-            <origin xyz="0 0 0" rpy="0 0 0"/>
-        </visual>
-        <collision>
-            <geometry>
-                <box size="${base_length + 2.0 * boundary_thickness} ${boundary_thickness} ${base_height + 2.0 * boundary_thickness}"/>
-            </geometry>
-            <origin xyz="0 0 0" rpy="0 0 0"/>
-        </collision>
-        <xacro:box_inertial mass="1.0" size="${base_length + 2.0 * boundary_thickness} ${boundary_thickness} ${base_height + 2.0 * boundary_thickness}" origin_xyz="0 0 0" origin_rpy="0 0 0"/>
-    </link>
-    <joint name="base_front_joint" type="fixed">
-        <parent link="base_link"/>
-        <child link="base_front_link"/>
-        <origin xyz="${+ (base_length + boundary_thickness) / 2.0} 0 0" rpy="0 0 0"/>
-    </joint>
-    <link name="base_front_link">
-        <visual>
-            <geometry>
-                <box size="${boundary_thickness} ${base_width + 2.0 * boundary_thickness} ${base_height + 2.0 * boundary_thickness}"/>
-            </geometry>
-            <material name="green"/>
-            <origin xyz="0 0 0" rpy="0 0 0"/>
-        </visual>
-        <collision>
-            <geometry>
-                <box size="${boundary_thickness} ${base_width + 2.0 * boundary_thickness} ${base_height + 2.0 * boundary_thickness}"/>
-            </geometry>
-            <origin xyz="0 0 0" rpy="0 0 0"/>
-        </collision>
-        <xacro:box_inertial mass="1.0" size="${boundary_thickness} ${base_width + 2.0 * boundary_thickness} ${base_height + 2.0 * boundary_thickness}" origin_xyz="0 0 0" origin_rpy="0 0 0"/>
-    </link>
-    <joint name="base_rear_joint" type="fixed">
-        <parent link="base_link"/>
-        <child link="base_rear_link"/>
-        <origin xyz="${- (base_length + boundary_thickness) / 2.0} 0 0" rpy="0 0 0"/>
-    </joint>
-    <link name="base_rear_link">
-        <visual>
-            <geometry>
-                <box size="${boundary_thickness} ${base_width + 2.0 * boundary_thickness} ${base_height + 2.0 * boundary_thickness}"/>
-            </geometry>
-            <material name="green"/>
-            <origin xyz="0 0 0" rpy="0 0 0"/>
-        </visual>
-        <collision>
-            <geometry>
-                <box size="${boundary_thickness} ${base_width + 2.0 * boundary_thickness} ${base_height + 2.0 * boundary_thickness}"/>
-            </geometry>
-            <origin xyz="0 0 0" rpy="0 0 0"/>
-        </collision>
-        <xacro:box_inertial mass="1.0" size="${boundary_thickness} ${base_width + 2.0 * boundary_thickness} ${base_height + 2.0 * boundary_thickness}" origin_xyz="0 0 0" origin_rpy="0 0 0"/>
-    </link>
-    <joint name="base_top_joint" type="fixed">
-        <parent link="base_link"/>
-        <child link="base_top_link"/>
-        <origin xyz="0 0 ${+ (base_height + boundary_thickness) / 2.0}" rpy="0 0 0"/>
-    </joint>
-    <link name="base_top_link">
-        <visual>
-            <geometry>
-                <box size="${base_length + 2.0 * boundary_thickness} ${base_width + 2.0 * boundary_thickness} ${boundary_thickness}"/>
-            </geometry>
-            <material name="green"/>
-            <origin xyz="0 0 0" rpy="0 0 0"/>
-        </visual>
-        <collision>
-            <geometry>
-                <box size="${base_length + 2.0 * boundary_thickness} ${base_width + 2.0 * boundary_thickness} ${boundary_thickness}"/>
-            </geometry>
-            <origin xyz="0 0 0" rpy="0 0 0"/>
-        </collision>
-        <xacro:box_inertial mass="1.0" size="${base_length + 2.0 * boundary_thickness} ${base_width + 2.0 * boundary_thickness} ${boundary_thickness}" origin_xyz="0 0 0" origin_rpy="0 0 0"/>
+        <xacro:box_inertial mass="5.0" size="${base_length} ${base_width} ${base_height}" origin_xyz="0 0 0" origin_rpy="0 0 0"/>
     </link>
     <joint name="base_left_wheel_joint" type="continuous">
         <parent link="base_link"/>
         <child link="left_wheel_link"/>
-        <origin xyz="0 ${+ (base_width - (wheel_length + epsilon)) / 2.0} ${- base_height / 2.0}" rpy="0 0 0"/>
+        <origin xyz="0 ${+ (base_width - wheel_length) / 2.0} ${- base_height / 2.0}" rpy="0 0 0"/>
         <axis xyz="0 1 0" />
     </joint>
@@ -170,5 +75,5 @@
         <parent link="base_link"/>
         <child link="right_wheel_link"/>
-        <origin xyz="0 ${- (base_width - (wheel_length + epsilon)) / 2.0 + epsilon} ${- base_height / 2.0}" rpy="0 0 0"/>
+        <origin xyz="0 ${- (base_width - wheel_length) / 2.0} ${- base_height / 2.0}" rpy="0 0 0"/>
         <axis xyz="0 1 0" />
     </joint>

File: src/mobile_robot_description/urdf/mobile_base_2.urdf.xacro (robot description, xacro)
@@ -16,8 +16,10 @@
                 </geometry>
                 <origin xyz="0 0 0" rpy="${pi / 2.0} 0 0" />
+                <material name="red" />
             </visual>
             <collision>
                 <geometry>
-                    <cylinder radius="${wheel_radius}" length="${wheel_length}"/>
+                    <!-- <cylinder radius="${wheel_radius}" length="${wheel_length}"/> -->
+                    <sphere radius="${wheel_radius}" />
                 </geometry>
                 <origin xyz="0 0 0" rpy="${pi / 2.0} 0 0" />
@@ -50,64 +52,97 @@
         <origin xyz="0 0 ${base_height / 2.0 + wheel_radius}" rpy="0 0 0"/>
     </joint>
-    <link name="base_link">
-        <!-- <visual>
-            <geometry>
-                <box size="${base_length} ${base_width} ${base_height}"/>
-            </geometry>
-            <material name="green"/>
-            <origin xyz="0 0 0" rpy="0 0 0"/>
-        </visual> -->
-        <visual>
-            <geometry>
-                <box size="${base_length + 2.0 * boundary_thickness} ${boundary_thickness} ${base_height + 2.0 * boundary_thickness}"/>
-            </geometry>
-            <material name="green"/>
-            <origin xyz="0 ${+ (base_width + boundary_thickness) / 2.0} 0" rpy="0 0 0"/>
-        </visual>
-        <collision>
-            <geometry>
-                <box size="${base_length + 2.0 * boundary_thickness} ${boundary_thickness} ${base_height + 2.0 * boundary_thickness}"/>
-            </geometry>
-            <origin xyz="0 ${+ (base_width + boundary_thickness) / 2.0} 0" rpy="0 0 0"/>
-        </collision>
-        <visual>
-            <geometry>
-                <box size="${base_length + 2.0 * boundary_thickness} ${boundary_thickness} ${base_height + 2.0 * boundary_thickness}"/>
-            </geometry>
-            <material name="green"/>
-            <origin xyz="0 ${- (base_width + boundary_thickness) / 2.0} 0" rpy="0 0 0"/>
-        </visual>
-        <collision>
-            <geometry>
-                <box size="${base_length + 2.0 * boundary_thickness} ${boundary_thickness} ${base_height + 2.0 * boundary_thickness}"/>
-            </geometry>
-            <origin xyz="0 ${- (base_width + boundary_thickness) / 2.0} 0" rpy="0 0 0"/>
-        </collision>
-        <visual>
-            <geometry>
-                <box size="${boundary_thickness} ${base_width + 2.0 * boundary_thickness} ${base_height + 2.0 * boundary_thickness}"/>
-            </geometry>
-            <material name="green"/>
-            <origin xyz="${+ (base_length + boundary_thickness) / 2.0} 0 0" rpy="0 0 0"/>
-        </visual>
-        <collision>
-            <geometry>
-                <box size="${boundary_thickness} ${base_width + 2.0 * boundary_thickness} ${base_height + 2.0 * boundary_thickness}"/>
-            </geometry>
-            <origin xyz="${+ (base_length + boundary_thickness) / 2.0} 0 0" rpy="0 0 0"/>
-        </collision>
-        <visual>
-            <geometry>
-                <box size="${boundary_thickness} ${base_width + 2.0 * boundary_thickness} ${base_height + 2.0 * boundary_thickness}"/>
-            </geometry>
-            <material name="green"/>
-            <origin xyz="${- (base_length + boundary_thickness) / 2.0} 0 0" rpy="0 0 0"/>
-        </visual>
-        <collision>
-            <geometry>
-                <box size="${boundary_thickness} ${base_width + 2.0 * boundary_thickness} ${base_height + 2.0 * boundary_thickness}"/>
-            </geometry>
-            <origin xyz="${- (base_length + boundary_thickness) / 2.0} 0 0" rpy="0 0 0"/>
-        </collision>
+    <link name="base_link" >
+        <xacro:box_inertial mass="1.0" size="${base_length} ${base_width} ${base_height}" origin_xyz="0 0 0" origin_rpy="0 0 0"/>
+    </link>
+    <joint name="base_left_joint" type="fixed">
+        <parent link="base_link"/>
+        <child link="base_left_link"/>
+        <origin xyz="0 ${+ (base_width + boundary_thickness) / 2.0} 0" rpy="0 0 0"/>
+    </joint>
+    <link name="base_left_link">
+        <visual>
+            <geometry>
+                <box size="${base_length + 2.0 * boundary_thickness} ${boundary_thickness} ${base_height + 2.0 * boundary_thickness}"/>
+            </geometry>
+            <material name="green"/>
+            <origin xyz="0 0 0" rpy="0 0 0"/>
+        </visual>
+        <collision>
+            <geometry>
+                <box size="${base_length + 2.0 * boundary_thickness} ${boundary_thickness} ${base_height + 2.0 * boundary_thickness}"/>
+            </geometry>
+            <origin xyz="0 0 0" rpy="0 0 0"/>
+        </collision>
+        <xacro:box_inertial mass="1.0" size="${base_length + 2.0 * boundary_thickness} ${boundary_thickness} ${base_height + 2.0 * boundary_thickness}" origin_xyz="0 0 0" origin_rpy="0 0 0"/>
+    </link>
+    <joint name="base_right_joint" type="fixed">
+        <parent link="base_link"/>
+        <child link="base_right_link"/>
+        <origin xyz="0 ${- (base_width + boundary_thickness) / 2.0} 0" rpy="0 0 0"/>
+    </joint>
+    <link name="base_right_link">
+        <visual>
+            <geometry>
+                <box size="${base_length + 2.0 * boundary_thickness} ${boundary_thickness} ${base_height + 2.0 * boundary_thickness}"/>
+            </geometry>
+            <material name="green"/>
+            <origin xyz="0 0 0" rpy="0 0 0"/>
+        </visual>
+        <collision>
+            <geometry>
+                <box size="${base_length + 2.0 * boundary_thickness} ${boundary_thickness} ${base_height + 2.0 * boundary_thickness}"/>
+            </geometry>
+            <origin xyz="0 0 0" rpy="0 0 0"/>
+        </collision>
+        <xacro:box_inertial mass="1.0" size="${base_length + 2.0 * boundary_thickness} ${boundary_thickness} ${base_height + 2.0 * boundary_thickness}" origin_xyz="0 0 0" origin_rpy="0 0 0"/>
+    </link>
+    <joint name="base_front_joint" type="fixed">
+        <parent link="base_link"/>
+        <child link="base_front_link"/>
+        <origin xyz="${+ (base_length + boundary_thickness) / 2.0} 0 0" rpy="0 0 0"/>
+    </joint>
+    <link name="base_front_link">
+        <visual>
+            <geometry>
+                <box size="${boundary_thickness} ${base_width + 2.0 * boundary_thickness} ${base_height + 2.0 * boundary_thickness}"/>
+            </geometry>
+            <material name="green"/>
+            <origin xyz="0 0 0" rpy="0 0 0"/>
+        </visual>
+        <collision>
+            <geometry>
+                <box size="${boundary_thickness} ${base_width + 2.0 * boundary_thickness} ${base_height + 2.0 * boundary_thickness}"/>
+            </geometry>
+            <origin xyz="0 0 0" rpy="0 0 0"/>
+        </collision>
+        <xacro:box_inertial mass="1.0" size="${boundary_thickness} ${base_width + 2.0 * boundary_thickness} ${base_height + 2.0 * boundary_thickness}" origin_xyz="0 0 0" origin_rpy="0 0 0"/>
+    </link>
+    <joint name="base_rear_joint" type="fixed">
+        <parent link="base_link"/>
+        <child link="base_rear_link"/>
+        <origin xyz="${- (base_length + boundary_thickness) / 2.0} 0 0" rpy="0 0 0"/>
+    </joint>
+    <link name="base_rear_link">
+        <visual>
+            <geometry>
+                <box size="${boundary_thickness} ${base_width + 2.0 * boundary_thickness} ${base_height + 2.0 * boundary_thickness}"/>
+            </geometry>
+            <material name="green"/>
+            <origin xyz="0 0 0" rpy="0 0 0"/>
+        </visual>
+        <collision>
+            <geometry>
+                <box size="${boundary_thickness} ${base_width + 2.0 * boundary_thickness} ${base_height + 2.0 * boundary_thickness}"/>
+            </geometry>
+            <origin xyz="0 0 0" rpy="0 0 0"/>
+        </collision>
+        <xacro:box_inertial mass="1.0" size="${boundary_thickness} ${base_width + 2.0 * boundary_thickness} ${base_height + 2.0 * boundary_thickness}" origin_xyz="0 0 0" origin_rpy="0 0 0"/>
+    </link>
+    <joint name="base_top_joint" type="fixed">
+        <parent link="base_link"/>
+        <child link="base_top_link"/>
+        <origin xyz="0 0 ${+ (base_height + boundary_thickness) / 2.0}" rpy="0 0 0"/>
+    </joint>
+    <link name="base_top_link">
         <visual>
             <geometry>
@@ -115,5 +150,5 @@
             </geometry>
             <material name="green"/>
-            <origin xyz="0 0 ${+ (base_height + boundary_thickness) / 2.0}" rpy="0 0 0"/>
+            <origin xyz="0 0 0" rpy="0 0 0"/>
         </visual>
         <collision>
@@ -121,7 +156,7 @@
                 <box size="${base_length + 2.0 * boundary_thickness} ${base_width + 2.0 * boundary_thickness} ${boundary_thickness}"/>
             </geometry>
-            <origin xyz="0 0 ${+ (base_height + boundary_thickness) / 2.0}" rpy="0 0 0"/>
-        </collision>
-        <xacro:box_inertial mass="5.0" size="${base_length + 2.0 * boundary_thickness} ${base_width + 2.0 * boundary_thickness} ${base_height + 2.0 * boundary_thickness}" origin_xyz="0 0 ${boundary_thickness}" origin_rpy="0 0 0"/>
+            <origin xyz="0 0 0" rpy="0 0 0"/>
+        </collision>
+        <xacro:box_inertial mass="1.0" size="${base_length + 2.0 * boundary_thickness} ${base_width + 2.0 * boundary_thickness} ${boundary_thickness}" origin_xyz="0 0 0" origin_rpy="0 0 0"/>
     </link>
     <joint name="base_left_wheel_joint" type="continuous">

File: src/mobile_robot_description/urdf/mobile_base_3.urdf.xacro (robot description, xacro)
@@ -12,14 +12,33 @@
                     <cylinder radius="${wheel_radius}" length="${wheel_length}"/>
                 </geometry>
-                <material name="red"/>
                 <origin xyz="0 0 0" rpy="${pi / 2.0} 0 0" />
+                <material name="red" />
             </visual>
-             <collision>
+            <collision>
                 <geometry>
-                    <cylinder radius="${wheel_radius}" length="${wheel_length}"/>
+                    <!-- <cylinder radius="${wheel_radius}" length="${wheel_length}"/> -->
+                    <sphere radius="${wheel_radius}" />
                 </geometry>
                 <origin xyz="0 0 0" rpy="${pi / 2.0} 0 0" />
             </collision>
-            <xacro:cylinder_inertial mass="1.0" radius="${wheel_radius}" length="${wheel_length}" origin_xyz="0 0 0" origin_rpy="${pi / 2.0} 0 0" />
+            <xacro:cylinder_inertial mass="0.5" radius="${wheel_radius}" length="${wheel_length}" origin_xyz="0 0 0" origin_rpy="${pi / 2.0} 0 0"/>
+        </link>
+    </xacro:macro>
+    <xacro:macro name="caster_wheel" params="prefix">
+        <link name="${prefix}_caster_wheel">
+            <visual>
+                <geometry>
+                    <sphere radius="${caster_wheel_radius}" />
+                </geometry>
+                <material name="gray" />
+                <origin xyz="0 0 0" rpy="0 0 0" />
+            </visual>
+            <collision>
+                <geometry>
+                    <sphere radius="${caster_wheel_radius}" />
+                </geometry>
+                <origin xyz="0 0 0" rpy="0 0 0" />
+            </collision>
+            <xacro:sphere_inertial mass="0.25" radius="${caster_wheel_radius}" origin_xyz="0 0 0" origin_rpy="0 0 0"/>
         </link>
     </xacro:macro>
