Commit message: add AMR meshes
On branch main
Your branch is up to date with 'origin/main'.

Changes to be committed:
	modified:   src/mobile_robot_bringup/launch/mobile_robot_gz_sim.launch.py
	modified:   src/mobile_robot_controller/config/mobile_robot_controllers.yaml
	modified:   src/mobile_robot_controller/launch/controller.launch.py
	modified:   src/mobile_robot_description/CMakeLists.txt
	modified:   src/mobile_robot_description/launch/display.launch.py
	new file:   src/mobile_robot_description/meshes/chasis.STL
	new file:   src/mobile_robot_description/meshes/wheel.STL
	new file:   src/mobile_robot_description/meshes/zed.STL
	new file:   src/mobile_robot_description/urdf/camera_1.urdf.xacro
	renamed:    src/mobile_robot_description/urdf/camera.urdf.xacro -> src/mobile_robot_description/urdf/camera_2.urdf.xacro
	modified:   src/mobile_robot_description/urdf/common_properties.urdf.xacro
	new file:   src/mobile_robot_description/urdf/depth_camera_1.urdf.xacro
	renamed:    src/mobile_robot_description/urdf/depth_camera.urdf.xacro -> src/mobile_robot_description/urdf/depth_camera_2.urdf.xacro
	renamed:    src/mobile_robot_description/urdf/imu.urdf.xacro -> src/mobile_robot_description/urdf/imu_1.urdf.xacro
	new file:   src/mobile_robot_description/urdf/imu_2.urdf.xacro
	modified:   src/mobile_robot_description/urdf/lidar.urdf.xacro
	new file:   src/mobile_robot_description/urdf/lidar_1.urdf.xacro
	new file:   src/mobile_robot_description/urdf/lidar_2.urdf.xacro
	new file:   src/mobile_robot_description/urdf/mobile_base.urdf.xacro
	modified:   src/mobile_robot_description/urdf/mobile_base_1.urdf.xacro
	modified:   src/mobile_robot_description/urdf/mobile_base_2.urdf.xacro
	modified:   src/mobile_robot_description/urdf/mobile_base_3.urdf.xacro
	modified:   src/mobile_robot_description/urdf/mobile_robot.urdf.xacro
	new file:   src/mobile_robot_description/urdf/zed_camera.urdf.xacro
	new file:   src/mobile_robot_description/urdf/zed_imu.urdf.xacro
	modified:   src/mobile_robot_description/worlds/Depot/model.sdf

File: src/mobile_robot_description/urdf/mobile_robot.urdf.xacro (robot description, xacro)
@@ -3,10 +3,14 @@
     <xacro:arg name="is_gz" default="true" />
     <xacro:include filename="common_properties.urdf.xacro"/>
-    <xacro:include filename="mobile_base_1.urdf.xacro" />
+    <!-- <xacro:include filename="mobile_base_1.urdf.xacro" />
+    <xacro:include filename="camera_1.urdf.xacro" />
+    <xacro:include filename="depth_camera_1.urdf.xacro" />
+    <xacro:include filename="imu_1.urdf.xacro" />
+    <xacro:include filename="lidar_1.urdf.xacro" /> -->
+    <xacro:include filename="mobile_base.urdf.xacro" />
+    <xacro:include filename="zed_camera.urdf.xacro" />
+    <xacro:include filename="zed_imu.urdf.xacro" />
+    <xacro:include filename="lidar.urdf.xacro" />
     <xacro:include filename="mobile_base_1_gazebo.urdf.xacro" />
     <xacro:include filename="mobile_base_1_ros2_control.urdf.xacro" />
-    <xacro:include filename="camera.urdf.xacro" />
-    <xacro:include filename="depth_camera.urdf.xacro" />
-    <xacro:include filename="imu.urdf.xacro" />
-    <xacro:include filename="lidar.urdf.xacro" />
 </robot>
