Commit message: add odometry
On branch main
Your branch is up to date with 'origin/main'.

Changes to be committed:
	new file:   frames_2025-11-22_02.23.18.gv
	new file:   frames_2025-11-22_02.23.18.pdf
	modified:   src/mobile_robot_bringup/config/gz_bridge.yaml
	modified:   src/mobile_robot_bringup/launch/mobile_robot_gz_sim.launch.py
	modified:   src/mobile_robot_controller/CMakeLists.txt
	modified:   src/mobile_robot_controller/config/mobile_robot_controllers.yaml
	new file:   src/mobile_robot_controller/include/mobile_robot_controller/noisy_odom.hpp
	new file:   src/mobile_robot_controller/include/mobile_robot_controller/perfect_odom.hpp
	modified:   src/mobile_robot_controller/include/mobile_robot_controller/simple_controller.hpp
	modified:   src/mobile_robot_controller/launch/controller.launch.py
	new file:   src/mobile_robot_controller/mobile_robot_controller/noisy_odom.py
	new file:   src/mobile_robot_controller/mobile_robot_controller/perfect_odom.py
	new file:   src/mobile_robot_controller/mobile_robot_controller/quaternion/__init__.py
	new file:   src/mobile_robot_controller/mobile_robot_controller/quaternion/quaternion.py
	modified:   src/mobile_robot_controller/mobile_robot_controller/simple_controller.py
	modified:   src/mobile_robot_controller/package.xml
	new file:   src/mobile_robot_controller/src/noisy_odom.cpp
	new file:   src/mobile_robot_controller/src/perfect_odom.cpp
	modified:   src/mobile_robot_controller/src/simple_controller.cpp
	modified:   src/mobile_robot_description/urdf/camera_1.urdf.xacro
	modified:   src/mobile_robot_description/urdf/depth_camera_1.urdf.xacro
	modified:   src/mobile_robot_description/urdf/imu_1.urdf.xacro
	modified:   src/mobile_robot_description/urdf/mobile_base_1.urdf.xacro
	modified:   src/mobile_robot_description/urdf/mobile_base_1_gazebo.urdf.xacro
	modified:   src/mobile_robot_description/urdf/mobile_base_gazebo.urdf.xacro
	modified:   src/mobile_robot_description/urdf/mobile_robot.urdf.xacro
	modified:   src/mobile_robot_description/urdf/zed_camera.urdf.xacro
	modified:   src/mobile_robot_description/urdf/zed_imu.urdf.xacro
	deleted:    src/mobile_robot_description/worlds/Depot/model copy.sdf
	modified:   src/mobile_robot_description/worlds/Depot/model.sdf
	new file:   src/mobile_robot_description/worlds/Depot/model_with_collision.sdf

File: src/mobile_robot_description/urdf/camera_1.urdf.xacro (robot description, xacro)
@@ -25,9 +25,18 @@
         <xacro:box_inertial mass="0.1" size="${camera_length} ${camera_width} ${camera_height}" origin_xyz="0 0 0" origin_rpy="0 0 0"/>
     </link>
-    <gazebo>
-        <plugin name="gz::sim::systems::Sensors" filename="gz-sim-sensors-system" >
-            <render_engine>ogre2</render_engine>
-        </plugin>
-    </gazebo>
+    <xacro:if value="$(arg is_gz)">
+        <gazebo>
+            <plugin name="gz::sim::systems::Sensors" filename="gz-sim-sensors-system" >
+                <render_engine>ogre2</render_engine>
+            </plugin>
+        </gazebo>
+    </xacro:if>
+    <xacro:unless value="$(arg is_gz)">
+        <gazebo>
+            <plugin name="ignition::gazebo::systems::Sensors" filename="ignition-gazebo-sensors-system" >
+                <render_engine>ogre2</render_engine>
+            </plugin>
+        </gazebo>
+    </xacro:unless>
     <gazebo reference="camera_link">
         <sensor name="camera" type="camera">

File: src/mobile_robot_description/urdf/depth_camera_1.urdf.xacro (robot description, xacro)
@@ -45,4 +45,5 @@
                     <stddev>0.007</stddev>
                 </noise>
+                <optical_fram_id>depth_camera_link</optical_fram_id>
             </depth_camera>
             <frame_id>depth_camera_link</frame_id>

File: src/mobile_robot_description/urdf/imu_1.urdf.xacro (robot description, xacro)
@@ -20,12 +20,61 @@
         <origin xyz="0 0 0" rpy="0 0 0"/>
     </joint>
-    <gazebo>
-        <plugin name="gz::sim::systems::Imu" filename="gz-sim-imu-system" />
-    </gazebo>
+    <xacro:if value="$(arg is_gz)">
+        <gazebo>
+            <plugin name="gz::sim::systems::Imu" filename="gz-sim-imu-system" />
+        </gazebo>
+    </xacro:if>
+    <xacro:unless value="$(arg is_gz)">
+        <gazebo>
+            <plugin name="ignition::gazebo::systems::Imu" filename="ignition-gazebo-imu-system" />
+        </gazebo>
+    </xacro:unless>
     <gazebo reference="imu_link">
         <sensor name="imu" type="imu">
-            <imu></imu>
+            <imu>
+                <angular_velocity>
+                    <x>
+                        <noise type="gaussian">
+                            <mean>0.0</mean>
+                            <stddev>2e-4</stddev>
+                        </noise>
+                    </x>
+                    <y>
+                        <noise type="gaussian">
+                            <mean>0.0</mean>
+                            <stddev>2e-4</stddev>
+                        </noise>
+                    </y>
+                    <z>
+                        <noise type="gaussian">
+                            <mean>0.0</mean>
+                            <stddev>2e-4</stddev>
+                        </noise>
+                    </z>
+                </angular_velocity>
+                <linear_acceleration>
+                    <x>
+                        <noise type="gaussian">
+                            <mean>0.0</mean>
+                            <stddev>2e-4</stddev>
+                        </noise>
+                    </x>
+                    <y>
+                        <noise type="gaussian">
+                            <mean>0.0</mean>
+                            <stddev>2e-4</stddev>
+                        </noise>
+                    </y>
+                    <z>
+                        <noise type="gaussian">
+                            <mean>0.0</mean>
+                            <stddev>2e-4</stddev>
+                        </noise>
+                    </z>
+                </linear_acceleration>
+            </imu>
             <always_on>1</always_on>
             <initialOrientationAsReference>false</initialOrientationAsReference>
+            <gz_frame_id>imu_link</gz_frame_id>
             <updateRate>100</updateRate>
             <visualize>true</visualize>

File: src/mobile_robot_description/urdf/mobile_base_1.urdf.xacro (robot description, xacro)
@@ -6,4 +6,5 @@
     <xacro:property name="wheel_radius" value="${base_height / 2.0}"/>
     <xacro:property name="wheel_length" value="${wheel_radius / 2.0}"/>
+    <xacro:property name="wheel_separation" value="0.35" />
     <xacro:property name="caster_wheel_radius" value="${wheel_radius / 2.0}" />
     <xacro:macro name="wheel_link" params="prefix">

File: src/mobile_robot_description/urdf/mobile_base_1_gazebo.urdf.xacro (robot description, xacro)
@@ -2,18 +2,26 @@
 <robot xmlns:xacro="http://www.ros.org/wiki/xacro">
     <gazebo reference="rear_left_caster_wheel">
-        <mu1 value="0.1"/>
-        <mu2 value="0.1"/>
+        <mu1 value="0.0001"/>
+        <mu2 value="0.0001"/>
     </gazebo>
     <gazebo reference="rear_right_caster_wheel">
-        <mu1 value="0.1"/>
-        <mu2 value="0.1"/>
+        <mu1 value="0.0001"/>
+        <mu2 value="0.0001"/>
     </gazebo>
     <gazebo reference="front_left_caster_wheel">
-        <mu1 value="0.1"/>
-        <mu2 value="0.1"/>
+        <mu1 value="0.0001"/>
+        <mu2 value="0.0001"/>
     </gazebo>
     <gazebo reference="front_right_caster_wheel">
-        <mu1 value="0.1"/>
-        <mu2 value="0.1"/>
+        <mu1 value="0.0001"/>
+        <mu2 value="0.0001"/>
+    </gazebo>
+    <gazebo reference="left_wheel_link">
+        <mu1 value="1000000"/>
+        <mu2 value="1000000"/>
+    </gazebo>
+    <gazebo reference="right_wheel_link">
+        <mu1 value="1000000"/>
+        <mu2 value="1000000"/>
     </gazebo>
     <xacro:if value="$(arg is_gz)" >
@@ -43,8 +51,8 @@
                 <parameters>$(find mobile_robot_controller)/config/mobile_robot_controllers.yaml</parameters>
                 <controller_manager_node_name>controller_manager</controller_manager_node_name>
-                <ros>
+                <!-- <ros>
                     <remapping>/diff_drive_base_controller/cmd_vel:=/cmd_vel</remapping>
                     <remapping>/diff_drive_base_controller/odom:=/odom</remapping>
-                </ros>
+                </ros> -->
             </plugin>
         </gazebo>
@@ -94,8 +102,8 @@
                 <parameters>$(find mobile_robot_controller)/config/mobile_robot_controllers.yaml</parameters>
                 <controller_manager_node_name>controller_manager</controller_manager_node_name>
-                <ros>
+                <!-- <ros>
                     <remapping>/diff_drive_base_controller/cmd_vel:=/cmd_vel</remapping>
                     <remapping>/diff_drive_base_controller/odom:=/odom</remapping>
-                </ros>
+                </ros> -->
             </plugin>
         </gazebo>

File: src/mobile_robot_description/urdf/mobile_base_gazebo.urdf.xacro (robot description, xacro)
@@ -43,8 +43,8 @@
                 <parameters>$(find mobile_robot_controller)/config/mobile_robot_controllers.yaml</parameters>
                 <controller_manager_node_name>controller_manager</controller_manager_node_name>
-                <ros>
+                <!-- <ros>
                     <remapping>/diff_drive_base_controller/cmd_vel:=/cmd_vel</remapping>
                     <remapping>/diff_drive_base_controller/odom:=/odom</remapping>
-                </ros>
+                </ros> -->
             </plugin>
         </gazebo>

File: src/mobile_robot_description/urdf/mobile_robot.urdf.xacro (robot description, xacro)
@@ -3,5 +3,5 @@
     <xacro:arg name="is_gz" default="true" />
     <xacro:include filename="common_properties.urdf.xacro"/>
-    <!-- <xacro:include filename="mobile_base_1.urdf.xacro" />
+    <xacro:include filename="mobile_base_1.urdf.xacro" />
     <xacro:include filename="camera_1.urdf.xacro" />
     <xacro:include filename="depth_camera_1.urdf.xacro" />
@@ -9,10 +9,10 @@
     <xacro:include filename="lidar_1.urdf.xacro" />
     <xacro:include filename="mobile_base_1_gazebo.urdf.xacro" />
-    <xacro:include filename="mobile_base_1_ros2_control.urdf.xacro" /> -->
-    <xacro:include filename="mobile_base.urdf.xacro" />
+    <xacro:include filename="mobile_base_1_ros2_control.urdf.xacro" />
+    <!-- <xacro:include filename="mobile_base.urdf.xacro" />
     <xacro:include filename="zed_camera.urdf.xacro" />
     <xacro:include filename="zed_imu.urdf.xacro" />
     <xacro:include filename="lidar.urdf.xacro" />
     <xacro:include filename="mobile_base_gazebo.urdf.xacro" />
-    <xacro:include filename="mobile_base_ros2_control.urdf.xacro" />
+    <xacro:include filename="mobile_base_ros2_control.urdf.xacro" /> -->
 </robot>

File: src/mobile_robot_description/urdf/zed_camera.urdf.xacro (robot description, xacro)
@@ -23,5 +23,5 @@
         </collision> -->
     </link>
-    <joint name="zed_camera_optical_joint" type="fixed">
+    <joint name="zed_camera_left_optical_joint" type="fixed">
         <parent link="zed_camera_link"/>
         <child link="zed_left_optical_frame"/>

File: src/mobile_robot_description/urdf/zed_imu.urdf.xacro (robot description, xacro)
@@ -28,12 +28,61 @@
         <origin xyz="0 0 0.02" rpy="0 0 0"/>
     </joint>
-    <gazebo>
-        <plugin name="gz::sim::systems::Imu" filename="gz-sim-imu-system" />
-    </gazebo>
+    <xacro:if value="$(arg is_gz)">
+        <gazebo>
+            <plugin name="gz::sim::systems::Imu" filename="gz-sim-imu-system" />
+        </gazebo>
+    </xacro:if>
+    <xacro:unless value="$(arg is_gz)">
+        <gazebo>
+            <plugin name="ignition::gazebo::systems::Imu" filename="ignition-gazebo-imu-system" />
+        </gazebo>
+    </xacro:unless>
     <gazebo reference="zed_imu_link">
         <sensor name="imu" type="imu">
-            <imu></imu>
+            <imu>
+                <angular_velocity>
+                    <x>
+                        <noise type="gaussian">
+                            <mean>0.0</mean>
+                            <stddev>2e-4</stddev>
+                        </noise>
+                    </x>
+                    <y>
+                        <noise type="gaussian">
+                            <mean>0.0</mean>
+                            <stddev>2e-4</stddev>
+                        </noise>
+                    </y>
+                    <z>
+                        <noise type="gaussian">
+                            <mean>0.0</mean>
+                            <stddev>2e-4</stddev>
+                        </noise>
+                    </z>
+                </angular_velocity>
+                <linear_acceleration>
+                    <x>
+                        <noise type="gaussian">
+                            <mean>0.0</mean>
+                            <stddev>2e-4</stddev>
+                        </noise>
+                    </x>
+                    <y>
+                        <noise type="gaussian">
+                            <mean>0.0</mean>
+                            <stddev>2e-4</stddev>
+                        </noise>
+                    </y>
+                    <z>
+                        <noise type="gaussian">
+                            <mean>0.0</mean>
+                            <stddev>2e-4</stddev>
+                        </noise>
+                    </z>
+                </linear_acceleration>
+            </imu>
             <always_on>1</always_on>
             <initialOrientationAsReference>false</initialOrientationAsReference>
+            <gz_frame_id>imu_link</gz_frame_id>
             <updateRate>100</updateRate>
             <visualize>true</visualize>
