Commit message: add ekf node from robot_localization pkg
On branch main
Your branch is up to date with 'origin/main'.

Changes to be committed:
	modified:   src/mobile_robot_bringup/launch/mobile_robot_gz_sim.launch.py
	modified:   src/mobile_robot_description/urdf/imu_1.urdf.xacro
	new file:   src/mobile_robot_localization/config/ekf_config.yaml
	modified:   src/mobile_robot_localization/launch/mobile_robot_localization.launch.py
	modified:   src/mobile_robot_localization/package.xml

File: src/mobile_robot_description/urdf/imu_1.urdf.xacro (robot description, xacro)
@@ -7,4 +7,5 @@
             </geometry>
             <material name="dark_gray" />
+            <origin xyz="0 0 0" rpy="0 0 0" />
         </visual>
         <collision>
@@ -12,4 +13,5 @@
                 <box size="0.05 0.05 0.05"/>
             </geometry>
+            <origin xyz="0 0 0" rpy="0 0 0" />
         </collision>
         <xacro:box_inertial mass="0.01" size="0.05 0.05 0.05" origin_xyz="0 0 0" origin_rpy="0 0 0"/>
